File: SOURCES/EAGLE/freeDSP.sch (EAGLE design)
At the start: 118 parts, among them IC1 24AA256P, IC3 AD8608R, Q1 12.288Mhz, Q2 2N7000, Q3 2N7000, Q4 2N7000, Q5 2N7000, T1 FZT751TA, X1 TOBU3, X2 TOBU3, X3 MKDSN1,5/2-5,08, X4 TOBU3, X5 TOBU3, X6 TOBU3, X7 TOBU3

Commit message: cleaned up the schematic and moved parts to different sheets
Parts:
- removed JP1: (no value), pinhead:PINHD-1X3
- R1: value 1k -> 1k 1%
- R2: value 18k -> 18k 1%
Connections:
- removed net N$40: R26.2, R30.2, R31.2, U$1.ADC0
- removed net N$7: C17.2, JP1.1, Q1.1
- new net ADC1: R28.2, R32.2, R33.2, U$1.ADC1
- net ADC0: now also R26.2, R30.2, R31.2, U$1.ADC0; no longer R28.2, R32.2, R33.2, U$1.ADC1
- net MCLK_IN: no longer JP1.3
- net N$10: now also C17.2, Q1.1; no longer JP1.2
Other:
- note added: "Power Supply"
- note removed: "<= 1% Tolerance!"
- note removed: "Jumper for Clock-Setting"
- note removed: "freeDSP 1.1 www.freedsp.cc"

Commit message: cleaned up sheet 0 and edited ADAU1701 to be smaller in the schematic
Other:
- note removed: "Crystal"
- moved on the sheet: C1, C10, C11, C12, C13, C15, C16, C17, C18, C19, C2, C20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
